File: placa_robot/placa_robot.kicad_sch (KiCad schematic)
At the start: 17 parts, among them IC1 MSP430FR2355TPT, J2 Conn_01x04, J3 Conn_02x04_Odd_Even, J4 conn_DFrobot, Y1 Crystal

Commit message: test_point
Parts:
- added J1: Conn_01x03, symbol Connector_Generic:Conn_01x03
- added TP1, TP10, TP11, TP12, TP2: TestPoint, symbol Connector:TestPoint
Connections:
- net +3.3V: now also TP1.1, TP10.1, TP2.1
- net GND: now also J1.3 (Pin_3)
- net SCL: now also TP11.1
- net SDA: now also TP12.1
Other:
- note added: "SBW"

Commit message: Conn Robot y pines
Parts:
- removed TP10: TestPoint, symbol Connector:TestPoint
Connections:
- net Sensor_Der is gone; now on an unnamed net: R10.2, RV2.2
- net Sensor_Izq is gone; now on an unnamed net: R9.2, RV1.2
- net P0: now also IC1.22 (P6.0/TB3.1)
- net P1: now also IC1.21 (P6.1/TB3.2)
- net P2: now also IC1.20 (P6.2/TB3.3)
- net P8: now also IC1.19 (P6.3/TB3.4)
- net P12: now reaches IC1.18 (P6.4/TB3.5)
- net P12: now also J4.12 (Pin_12)
Other:
- note added: "Microcontrolador | si LCDs | si Cuarzo | si️ LDR | si Sensor Ultra so | no Joystick | si WIFI | Si conexion con robot | si detector de programación | si asignación de los pines | no"
- note removed: "Microcontrolador | si LCDs | no Cuarzo | si️ LDR | si Sensor Ultraso | No Joystick | si WIFI | Si conexion con robot | no detector de programación | no asignación de los pines | no"

Commit message: SBW reset
Parts:
- added C5: 1nF, symbol Device:C
- added R16: 47k, symbol Device:R
- added SW1: SW_Push, symbol Switch:SW_Push
Connections:
- net +3.3V: now also R16.1
- net GND: now also C5.1, SW1.1
- net at IC1.4 (TEST/SBWTCK): now also J1.1 (Pin_1)
- net at IC1.5 (~{RST}/NMI/SBWTDIO): now also J1.2 (Pin_2), C5.2, R16.2, SW1.2
Other:
- note added: "Microcontrolador | si LCDs | si Cuarzo | si️ LDR | si Sensor Ultra so | si Joystick | si WIFI | Si conexion con robot | si detector de programación | si asignación de los pines | no"
- note removed: "Microcontrolador | si LCDs | si Cuarzo | si️ LDR | si Sensor Ultra so | no Joystick | si WIFI | Si conexion con robot | si detector de programación | si asignación de los pines | no"
- moved on the sheet: C2, C4, J1, Y1

Commit message: Connectar Joystick
Connections:
- net Joystick_Boton: now also IC1.37 (P3.5/OA3O)
- net Joystick_Down: now also IC1.44 (P3.3/OA2+)
- net Joystick_Left: now also IC1.45 (P3.2/OA2-)
- net Joystick_Right: now also IC1.46 (P3.1/OA2O)
- net Joystick_Up: now also IC1.38 (P3.4/SMCLK)
Changed lines of the file:
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@@
+	(wire
+		(pts
+			(xy 199.39 59.69) (xy 199.39 76.2)
+		)
+		(stroke
+			(width 0)
+			(type default)
+		)
+	)
 	(wire
 		(pts
@@
 	(wire
 		(pts
+			(xy 214.63 63.5) (xy 214.63 76.2)
+		)
+		(stroke
+			(width 0)
+			(type default)
+		)
+	)
+	(wire
+		(pts
 			(xy 214.63 259.08) (xy 214.63 273.05)
 		)
@@
 	(wire
 		(pts
+			(xy 218.44 59.69) (xy 199.39 59.69)
+		)
+		(stroke
+			(width 0)
+			(type default)
+		)
+	)
+	(wire
+		(pts
 			(xy 274.32 152.4) (xy 274.32 149.86)
 		)
@@
 	(wire
 		(pts
+			(xy 218.44 63.5) (xy 214.63 63.5)
+		)
+		(stroke
+			(width 0)
+			(type default)
+		)
+	)
+	(wire
+		(pts
 			(xy 267.97 147.32) (xy 275.59 147.32)
 		)
@@
 	(wire
 		(pts
+			(xy 218.44 55.88) (xy 196.85 55.88)
+		)
+		(stroke
+			(width 0)
+			(type default)
+		)
+	)
+	(wire
+		(pts
 			(xy 130.81 134.62) (xy 138.43 134.62)
 		)
@@
 	(wire
 		(pts
+			(xy 196.85 55.88) (xy 196.85 76.2)
+		)
+		(stroke
+			(width 0)
+			(type default)
+		)
+	)
+	(wire
+		(pts
 			(xy 83.82 76.2) (xy 78.74 76.2)
 		)
@@
 	(wire
 		(pts
+			(xy 217.17 67.31) (xy 217.17 76.2)
+		)
+		(stroke
+			(width 0)
+			(type default)
+		)
+	)
+	(wire
+		(pts
 			(xy 54.61 220.98) (xy 54.61 219.71)
 		)
@@
 	(wire
 		(pts
+			(xy 194.31 52.07) (xy 194.31 76.2)
+		)
+		(stroke
+			(width 0)
+			(type default)
+		)
+	)
+	(wire
+		(pts
 			(xy 214.63 273.05) (xy 267.97 273.05)
 		)
@@
 	(wire
 		(pts
+			(xy 218.44 52.07) (xy 194.31 52.07)
+		)
+		(stroke
+			(width 0)
+			(type default)
+		)
+	)
+	(wire
+		(pts
 			(xy 189.23 241.3) (xy 189.23 200.66)
 		)
@@
 		(pts
 			(xy 204.47 76.2) (xy 204.47 64.77)
+		)
+		(stroke
+			(width 0)
+			(type default)
+		)
+	)
+	(wire
+		(pts
+			(xy 218.44 67.31) (xy 217.17 67.31)
 		)
 		(stroke
@@
 	(global_label "Joystick_Left"
 		(shape input)
-		(at 295.91 135.89 0)
+		(at 218.44 55.88 0)
 		(fields_autoplaced yes)
 		(effects
@@
 		)
 		(property "Intersheetrefs" "${INTERSHEET_REFS}"
-			(at 310.9904 135.89 0)
+			(at 233.5204 55.88 0)
 			(effects
 				(font
@@
 	(global_label "Joystick_Boton"
 		(shape input)
-		(at 295.91 143.51 0)
+		(at 218.44 67.31 0)
 		(fields_autoplaced yes)
 		(effects
@@
 		)
 		(property "Intersheetrefs" "${INTERSHEET_REFS}"
-			(at 312.865 143.51 0)
+			(at 235.395 67.31 0)
 			(effects
 				(font
@@
 	(global_label "Joystick_Up"
 		(shape input)
-		(at 295.91 140.97 0)
+		(at 218.44 63.5 0)
 		(fields_autoplaced yes)
 		(effects
@@
 		)
 		(property "Intersheetrefs" "${INTERSHEET_REFS}"
-			(at 309.9018 140.97 0)
+			(at 232.4318 63.5 0)
 			(effects
 				(font
@@
 	(global_label "Joystick_Right"
 		(shape input)
-		(at 295.91 133.35 0)
+		(at 218.44 52.07 0)
 		(fields_autoplaced yes)
 		(effects
@@
 		)
 		(property "Intersheetrefs" "${INTERSHEET_REFS}"
-			(at 312.3208 133.35 0)
+			(at 234.8508 52.07 0)
 			(effects
 				(font
@@
 	(global_label "Joystick_Down"
 		(shape input)
-		(at 295.91 138.43 0)
+		(at 218.44 59.69 0)
 		(fields_autoplaced yes)
 		(effects
@@
 		)
 		(property "Intersheetrefs" "${INTERSHEET_REFS}"
-			(at 312.3208 138.43 0)
+			(at 234.8508 59.69 0)
 			(effects
 				(font

Commit message: test point
Parts:
- added TP10, TP13: TestPoint, symbol Connector:TestPoint
Connections:
- net U0RXD: now also TP10.1
- net U0TXD: now also TP13.1
Changed lines of the file:
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@@
 	)
 	(junction
+		(at 353.06 99.06)
+		(diameter 0)
+		(color 0 0 0 0)
+	)
+	(junction
 		(at 82.55 226.06)
 		(diameter 0)
@@
 	)
 	(junction
+		(at 327.66 87.63)
+		(diameter 0)
+		(color 0 0 0 0)
+	)
+	(junction
 		(at 127 142.24)
 		(diameter 0)
@@
 	(wire
 		(pts
-			(xy 346.71 95.25) (xy 351.79 95.25)
-		)
-		(stroke
-			(width 0)
-			(type default)
-		)
-	)
-	(wire
-		(pts
 			(xy 127 143.51) (xy 127 142.24)
 		)
@@
 	(wire
 		(pts
+			(xy 353.06 104.14) (xy 353.06 99.06)
+		)
+		(stroke
+			(width 0)
+			(type default)
+		)
+	)
+	(wire
+		(pts
 			(xy 214.63 273.05) (xy 267.97 273.05)
 		)
@@
 	(wire
 		(pts
-			(xy 330.2 87.63) (xy 334.01 87.63)
+			(xy 325.12 87.63) (xy 327.66 87.63)
 		)
 		(stroke
@@
 	(wire
 		(pts
+			(xy 327.66 82.55) (xy 327.66 87.63)
+		)
+		(stroke
+			(width 0)
+			(type default)
+		)
+	)
+	(wire
+		(pts
+			(xy 353.06 99.06) (xy 353.06 95.25)
+		)
+		(stroke
+			(width 0)
+			(type default)
+		)
+	)
+	(wire
+		(pts
 			(xy 111.76 142.24) (xy 116.84 142.24)
 		)
@@
 	(wire
 		(pts
+			(xy 353.06 95.25) (xy 346.71 95.25)
+		)
+		(stroke
+			(width 0)
+			(type default)
+		)
+	)
+	(wire
+		(pts
 			(xy 262.89 257.81) (xy 262.89 212.09)
 		)
@@
 	(wire
 		(pts
+			(xy 353.06 99.06) (xy 359.41 99.06)
+		)
+		(stroke
+			(width 0)
+			(type default)
+		)
+	)
+	(wire
+		(pts
 			(xy 119.38 234.95) (xy 119.38 241.3)
 		)
@@
 	(wire
 		(pts
+			(xy 327.66 87.63) (xy 334.01 87.63)
+		)
+		(stroke
+			(width 0)
+			(type default)
+		)
+	)
+	(wire
+		(pts
 			(xy 78.74 67.31) (xy 78.74 68.58)
 		)
@@
 	(global_label "U0RXD"
 		(shape input)
-		(at 330.2 87.63 180)
+		(at 325.12 87.63 180)
 		(fields_autoplaced yes)
 		(effects
@@
 		)
 		(property "Intersheetrefs" "${INTERSHEET_REFS}"
-			(at 320.9253 87.63 0)
+			(at 315.8453 87.63 0)
 			(effects
 				(font
@@
 	(global_label "U0TXD"
 		(shape input)
-		(at 351.79 95.25 0)
+		(at 353.06 104.14 0)
 		(fields_autoplaced yes)
 		(effects
@@
 		)
 		(property "Intersheetrefs" "${INTERSHEET_REFS}"
-			(at 360.7623 95.25 0)
+			(at 362.0323 104.14 0)
 			(effects
 				(font
@@
 	)
 	(symbol
+		(lib_id "Connector:TestPoint")
+		(at 359.41 99.06 0)
+		(mirror y)
+		(unit 1)
+		(exclude_from_sim no)
+		(in_bom yes)
+		(on_board yes)
+		(dnp no)
+		(property "Reference" "TP13"
+			(at 367.284 95.25 0)
+			(effects
+				(font
+					(size 1.27 1.27)
+				)
+				(justify left)
+			)
+		)
+		(property "Value" "TestPoint"
+			(at 370.586 97.282 0)
+			(effects
+				(font
+					(size 1.27 1.27)
+				)
+				(justify left)
+			)
+		)
+		(property "Footprint" ""
+			(at 354.33 99.06 0)
+			(effects
+				(font
+					(size 1.27 1.27)
+				)
+				(hide yes)
+			)
+		)
+		(property "Datasheet" "~"
+			(at 354.33 99.06 0)
+			(effects
+				(font
+					(size 1.27 1.27)
+				)
+				(hide yes)
+			)
+		)
+		(property "Description" "test point"
+			(at 359.41 99.06 0)
+			(effects
+				(font
+					(size 1.27 1.27)
+				)
+				(hide yes)
+			)
+		)
+		(pin "1"
+		)
+		(instances
+			(project "placa_robot"
+				(path "/8aa50d15-d96a-41b3-aa5f-664bff39212d"
+					(reference "TP13")
+					(unit 1)
+				)
+			)
+		)
+	)
+	(symbol
 		(lib_id "power:GND")
 		(at 46.99 229.87 0)
@@
 					(unit 1)
 				)
+			)
+		)
+	)
+	(symbol
+		(lib_id "Connector:TestPoint")
+		(at 327.66 82.55 0)
+		(unit 1)
+		(exclude_from_sim no)
+		(in_bom yes)
+		(on_board yes)
+		(dnp no)
+		(property "Reference" "TP10"
+			(at 319.786 78.74 0)
+			(effects
+				(font
+					(size 1.27 1.27)
+				)
+				(justify left)
+			)
+		)
+		(property "Value" "TestPoint"
+			(at 316.484 80.772 0)
+			(effects
+				(font
+					(size 1.27 1.27)
+				)
+				(justify left)
+			)
+		)
+		(property "Footprint" ""
+			(at 332.74 82.55 0)
+			(effects
+				(font
+					(size 1.27 1.27)
+				)
+				(hide yes)
+			)
+		)
+		(property "Datasheet" "~"
+			(at 332.74 82.55 0)
+			(effects
+				(font
+					(size 1.27 1.27)
+				)
+				(hide yes)
+			)
+		)
+		(property "Description" "test point"
+			(at 327.66 82.55 0)
+			(effects
+				(font
+					(size 1.27 1.27)
+				)
+				(hide yes)
+			)
+		)
+		(pin "1"
+		)
+		(instances
+			(project "placa_robot"
+				(path "/8aa50d15-d96a-41b3-aa5f-664bff39212d"
+					(reference "TP10")
+					(unit 1)
+				)

Commit message: hola
Connections:
- net RST(LCD) is gone; now on an unnamed net: LCD1.5 (RST)
Changed lines of the file:
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@@
 	(wire
 		(pts
+			(xy 199.39 200.66) (xy 199.39 205.74)
+		)
+		(stroke
+			(width 0)
+			(type default)
+		)
+	)
+	(wire
+		(pts
+			(xy 113.03 205.74) (xy 199.39 205.74)
+		)
+		(stroke
+			(width 0)
+			(type default)
+		)
+	)
+	(wire
+		(pts
 			(xy 134.62 144.78) (xy 138.43 144.78)
 		)
@@
 	(wire
 		(pts
+			(xy 203.2 260.35) (xy 203.2 259.08)
+		)
+		(stroke
+			(width 0)
+			(type default)
+		)
+	)
+	(wire
+		(pts
 			(xy 265.43 255.27) (xy 265.43 270.51)
 		)
@@
 	(wire
 		(pts
+			(xy 69.85 219.71) (xy 69.85 236.22)
+		)
+		(stroke
+			(width 0)
+			(type default)
+		)
+	)
+	(wire
+		(pts
 			(xy 214.63 63.5) (xy 214.63 76.2)
 		)
@@
 	(wire
 		(pts
+			(xy 69.85 236.22) (xy 113.03 236.22)
+		)
+		(stroke
+			(width 0)
+			(type default)
+		)
+	)
+	(wire
+		(pts
 			(xy 274.32 142.24) (xy 275.59 142.24)
 		)
@@
 	(wire
 		(pts
-			(xy 274.32 138.43) (xy 274.32 142.24)
+			(xy 274.32 135.89) (xy 274.32 142.24)
 		)
 		(stroke
@@
 	(wire
 		(pts
+			(xy 113.03 236.22) (xy 113.03 205.74)
+		)
+		(stroke
+			(width 0)
+			(type default)
+		)
+	)
+	(wire
+		(pts
 			(xy 119.38 241.3) (xy 167.64 241.3)
 		)
@@
 	(wire
 		(pts
+			(xy 231.14 243.84) (xy 231.14 246.38)
+		)
+		(stroke
+			(width 0)
+			(type default)
+		)
+	)
+	(wire
+		(pts
 			(xy 134.62 132.08) (xy 138.43 132.08)
 		)
@@
 		)
 	)
-	(global_label "RST(LCD)"
-		(shape bidirectional)
-		(at 69.85 219.71 270)
-		(fields_autoplaced yes)
-		(effects
-			(font
-				(size 1.27 1.27)
-			)
-			(justify right)
-		)
-		(property "Intersheetrefs" "${INTERSHEET_REFS}"
-			(at 69.85 232.5151 90)
-			(effects
-				(font
-					(size 1.27 1.27)
-				)
-				(justify right)
-				(hide yes)
-			)
-		)
-	)
 	(symbol
 		(lib_id "power:GND")
@@
 	(symbol
 		(lib_id "power:+3.3V")
-		(at 274.32 138.43 0)
+		(at 274.32 135.89 0)
 		(unit 1)
 		(exclude_from_sim no)
@@
 		(fields_autoplaced yes)
 		(property "Reference" "#PWR021"
-			(at 274.32 142.24 0)
+			(at 274.32 139.7 0)
 			(effects
 				(font
@@
 		)
 		(property "Value" "+3.3V"
-			(at 274.32 133.35 0)
+			(at 274.32 130.81 0)
 			(effects
 				(font
@@
 		)
 		(property "Footprint" ""
-			(at 274.32 138.43 0)
+			(at 274.32 135.89 0)
 			(effects
 				(font
@@
 		)
 		(property "Datasheet" ""
-			(at 274.32 138.43 0)
+			(at 274.32 135.89 0)
 			(effects
 				(font
@@
 		)
 		(property "Description" "Power symbol creates a global label with name \"+3.3V\""
-			(at 274.32 138.43 0)
+			(at 274.32 135.89 0)
 			(effects
 				(font
@@
 		(on_board yes)
 		(dnp no)
-		(fields_autoplaced yes)
 		(property "Reference" "J4"
 			(at 207.01 251.4599 90)
@@
 		)
 		(property "Value" "conn_DFrobot"
-			(at 207.01 253.9999 90)
+			(at 200.914 253.238 90)
 			(effects
 				(font
@@
 	(symbol
 		(lib_id "power:GND")
-		(at 203.2 259.08 0)
+		(at 203.2 260.35 0)
 		(unit 1)
 		(exclude_from_sim no)
@@
 		(fields_autoplaced yes)
 		(property "Reference" "#PWR05"
-			(at 203.2 265.43 0)
+			(at 203.2 266.7 0)
 			(effects
 				(font
@@
 		)
 		(property "Value" "GND"
-			(at 203.2 264.16 0)
+			(at 203.2 265.43 0)
 			(effects
 				(font
@@
 		)
 		(property "Footprint" ""
-			(at 203.2 259.08 0)
+			(at 203.2 260.35 0)
 			(effects
 				(font
@@
 		)
 		(property "Datasheet" ""
-			(at 203.2 259.08 0)
+			(at 203.2 260.35 0)
 			(effects
 				(font
@@
 		)
 		(property "Description" "Power symbol creates a global label with name \"GND\" , ground"
-			(at 203.2 259.08 0)
+			(at 203.2 260.35 0)
 			(effects
 				(font
@@
 	(symbol
 		(lib_id "power:+3.3V")
-		(at 231.14 246.38 0)
+		(at 231.14 243.84 0)
 		(unit 1)
 		(exclude_from_sim no)
@@
 		(fields_autoplaced yes)
 		(property "Reference" "#PWR023"
-			(at 231.14 250.19 0)
+			(at 231.14 247.65 0)
 			(effects
 				(font
@@
 		)
 		(property "Value" "+3.3V"
-			(at 231.14 241.3 0)
+			(at 231.14 238.76 0)
 			(effects
 				(font
@@
 		)
 		(property "Footprint" ""
-			(at 231.14 246.38 0)
+			(at 231.14 243.84 0)
 			(effects
 				(font
@@
 		)
 		(property "Datasheet" ""
-			(at 231.14 246.38 0)
+			(at 231.14 243.84 0)
 			(effects
 				(font
@@
 		)
 		(property "Description" "Power symbol creates a global label with name \"+3.3V\""
-			(at 231.14 246.38 0)
+			(at 231.14 243.84 0)
 			(effects
 				(font

Commit message: wifi
Connections:
- net U0RXD is gone; now on an unnamed net: J3.1 (Pin_1), TP10.1
- net U0TXD is gone; now on an unnamed net: J3.8 (Pin_8), TP13.1
Other:
- note removed: "Microcontrolador | si LCDs | si Cuarzo | si️ LDR | si Sensor Ultra so | si Joystick | si WIFI | Si conexion con robot | si detector de programación | si asignación de los pines | no"
- moved on the sheet: C2, C3, C4, C5, IC1, J1, J2, J3, J4, JP1, LCD1, R10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
