File: placa_robot/placa_robot.kicad_sch (KiCad schematic)
At the start: 37 parts, among them IC1 MSP430FR2355TPT, J1 Conn_01x03, J3 Conn_02x04_Odd_Even, J4 conn_DFrobot, SW1 SW_Push, U1 LM324, Y1 Crystal

Commit message: Layout
Parts:
- R10, R9: footprint Resistor_SMD:R_0805_2012Metric_Pad1.20x1.40mm_HandSolder -> Connector_PinHeader_2.54mm:PinHeader_1x02_P2.54mm_Horizontal
- S2: footprint THB001P -> (none)
Changed lines of the file:
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@@
 			)
 		)
-		(property "Footprint" "Resistor_SMD:R_0805_2012Metric_Pad1.20x1.40mm_HandSolder"
+		(property "Footprint" "Connector_PinHeader_2.54mm:PinHeader_1x02_P2.54mm_Horizontal"
 			(at 72.39 48.26 90)
 			(effects
@@
 			)
 		)
-		(property "Footprint" "Resistor_SMD:R_0805_2012Metric_Pad1.20x1.40mm_HandSolder"
+		(property "Footprint" "Connector_PinHeader_2.54mm:PinHeader_1x02_P2.54mm_Horizontal"
 			(at 90.17 48.26 90)
 			(effects
@@
 			)
 		)
-		(property "Footprint" "THB001P"
+		(property "Footprint" ""
 			(at 367.03 225.73 0)
 			(effects

Commit message: Progreso actual Layout y errores
Parts:
- LCD1: footprint Connector_PinHeader_2.54mm:PinHeader_1x02_P2.54mm_Horizontal -> MiSE:LCD_2x16_I2C(Midas)
Connections:
- net P0: now also IC1.18 (P6.4/TB3.5); no longer IC1.22 (P6.0/TB3.1)
- net P1: now also IC1.19 (P6.3/TB3.4); no longer IC1.21 (P6.1/TB3.2)
- net P12: now also IC1.22 (P6.0/TB3.1); no longer IC1.18 (P6.4/TB3.5)
- net P8: now also IC1.21 (P6.1/TB3.2); no longer IC1.19 (P6.3/TB3.4)
Changed lines of the file:
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@@
 	(wire
 		(pts
-			(xy 193.04 199.39) (xy 193.04 218.44)
-		)
-		(stroke
-			(width 0)
-			(type default)
-		)
-	)
-	(wire
-		(pts
 			(xy 215.9 257.81) (xy 222.25 257.81)
 		)
@@
 	(wire
 		(pts
-			(xy 200.66 199.39) (xy 200.66 210.82)
+			(xy 90.17 160.02) (xy 95.25 160.02)
 		)
 		(stroke
@@
 	(wire
 		(pts
-			(xy 90.17 160.02) (xy 95.25 160.02)
+			(xy 386.08 74.93) (xy 386.08 80.01)
 		)
 		(stroke
@@
 	(wire
 		(pts
-			(xy 386.08 74.93) (xy 386.08 80.01)
+			(xy 198.12 199.39) (xy 198.12 213.36)
 		)
 		(stroke
@@
 	(wire
 		(pts
+			(xy 195.58 210.82) (xy 195.58 199.39)
+		)
+		(stroke
+			(width 0)
+			(type default)
+		)
+	)
+	(wire
+		(pts
 			(xy 95.25 147.32) (xy 90.17 147.32)
 		)
@@
 	(wire
 		(pts
-			(xy 198.12 199.39) (xy 198.12 213.36)
+			(xy 193.04 208.28) (xy 251.46 208.28)
 		)
 		(stroke
@@
 	(wire
 		(pts
-			(xy 203.2 199.39) (xy 203.2 208.28)
-		)
-		(stroke
-			(width 0)
-			(type default)
-		)
-	)
-	(wire
-		(pts
 			(xy 336.55 124.46) (xy 336.55 135.89)
 		)
@@
 	(wire
 		(pts
-			(xy 259.08 215.9) (xy 195.58 215.9)
+			(xy 259.08 215.9) (xy 200.66 215.9)
 		)
 		(stroke
@@
 	(wire
 		(pts
-			(xy 95.25 116.84) (xy 105.41 116.84)
+			(xy 195.58 210.82) (xy 254 210.82)
 		)
 		(stroke
@@
 	(wire
 		(pts
-			(xy 128.27 151.13) (xy 128.27 237.49)
+			(xy 95.25 116.84) (xy 105.41 116.84)
 		)
 		(stroke
@@
 	(wire
 		(pts
-			(xy 367.03 93.98) (xy 367.03 77.47)
+			(xy 128.27 151.13) (xy 128.27 237.49)
 		)
 		(stroke
@@
 	(wire
 		(pts
-			(xy 336.55 143.51) (xy 336.55 135.89)
+			(xy 367.03 93.98) (xy 367.03 77.47)
 		)
 		(stroke
@@
 	(wire
 		(pts
-			(xy 246.38 254) (xy 256.54 254)
+			(xy 336.55 143.51) (xy 336.55 135.89)
 		)
 		(stroke
@@
 	(wire
 		(pts
-			(xy 60.96 234.95) (xy 104.14 234.95)
+			(xy 246.38 254) (xy 256.54 254)
 		)
 		(stroke
@@
 	(wire
 		(pts
-			(xy 327.66 77.47) (xy 325.12 77.47)
+			(xy 60.96 234.95) (xy 104.14 234.95)
 		)
 		(stroke
@@
 	(wire
 		(pts
-			(xy 254 210.82) (xy 200.66 210.82)
+			(xy 327.66 77.47) (xy 325.12 77.47)
 		)
 		(stroke
@@
 	(wire
 		(pts
-			(xy 195.58 215.9) (xy 195.58 199.39)
-		)
-		(stroke
-			(width 0)
-			(type default)
-		)
-	)
-	(wire
-		(pts
 			(xy 205.74 60.96) (xy 304.8 60.96)
 		)
@@
 	(wire
 		(pts
+			(xy 200.66 199.39) (xy 200.66 215.9)
+		)
+		(stroke
+			(width 0)
+			(type default)
+		)
+	)
+	(wire
+		(pts
 			(xy 64.77 224.79) (xy 73.66 224.79)
 		)
@@
 	(wire
 		(pts
+			(xy 193.04 199.39) (xy 193.04 208.28)
+		)
+		(stroke
+			(width 0)
+			(type default)
+		)
+	)
+	(wire
+		(pts
 			(xy 76.2 50.8) (xy 76.2 57.15)
 		)
@@
 	(wire
 		(pts
-			(xy 261.62 218.44) (xy 193.04 218.44)
+			(xy 261.62 218.44) (xy 203.2 218.44)
 		)
 		(stroke
@@
 	(wire
 		(pts
-			(xy 251.46 208.28) (xy 203.2 208.28)
+			(xy 304.8 60.96) (xy 304.8 80.01)
 		)
 		(stroke
@@
 	(wire
 		(pts
-			(xy 304.8 60.96) (xy 304.8 80.01)
+			(xy 386.08 80.01) (xy 403.86 80.01)
 		)
 		(stroke
@@
 	(wire
 		(pts
-			(xy 386.08 80.01) (xy 403.86 80.01)
+			(xy 259.08 271.78) (xy 259.08 251.46)
 		)
 		(stroke
@@
 	(wire
 		(pts
-			(xy 259.08 271.78) (xy 259.08 251.46)
+			(xy 80.01 160.02) (xy 80.01 165.1)
 		)
 		(stroke
@@
 	(wire
 		(pts
-			(xy 80.01 160.02) (xy 80.01 165.1)
+			(xy 302.26 146.05) (xy 302.26 63.5)
 		)
 		(stroke
@@
 	(wire
 		(pts
-			(xy 302.26 146.05) (xy 302.26 63.5)
+			(xy 203.2 199.39) (xy 203.2 218.44)
 		)
 		(stroke
@@
 			)
 		)
-		(property "Footprint" "Connector_PinHeader_2.54mm:PinHeader_1x02_P2.54mm_Horizontal"
+		(property "Footprint" "MiSE:LCD_2x16_I2C(Midas)"
 			(at 55.88 195.58 0)
 			(effects

Commit message: Cambios layout
Parts:
- added J2: Conn_01x01, Connector_PinHeader_2.54mm:PinHeader_1x01_P2.54mm_Vertical, symbol Connector_Generic:Conn_01x01
- S2: footprint (none) -> MiSE:THB001P
- SW1: footprint (none) -> Button_Switch_THT:SW_PUSH_6mm
Connections:
- net DOWN: now also IC1.46 (P3.1/OA2O); no longer IC1.45 (P3.2/OA2-)
- net GND: now also J2.1 (Pin_1)
- net Photo1: now also IC1.43 (P5.0/TB2.1/MFM.RX/A8); no longer IC1.42 (P5.1/TB2.2/MFM.TX/A9)
- net Photo2: now also IC1.42 (P5.1/TB2.2/MFM.TX/A9); no longer IC1.43 (P5.0/TB2.1/MFM.RX/A8)
- net UP: now also IC1.45 (P3.2/OA2-); no longer IC1.46 (P3.1/OA2O)
Other:
- note added: "Un connector a gnd que lo necesitaremos, cuando usemos los test Points"

Commit message: cambio layout
Connections:
- net +3.3V: no longer JP1.1 (A), LCD1.6 (A)
- net WIFI_RXD: now also IC1.23 (P4.3/UCA1TXD/UCA1SIMO/~{UCA1TXD}); no longer IC1.24 (P4.2/UCA1RXD/UCA1SOMI/~{UCA1RXD})
- net WIFI_TXD: now also IC1.24 (P4.2/UCA1RXD/UCA1SOMI/~{UCA1RXD}); no longer IC1.23 (P4.3/UCA1TXD/UCA1SIMO/~{UCA1TXD})
- net XIN: now also C2.2, Y1.1; no longer C4.2, Y1.2
- net XOUT: now also C4.2, Y1.2; no longer C2.2, Y1.1
- new net: JP1.1 (A), LCD1.6 (A)
Changed lines of the file:
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@@
+	)
+	(junction
+		(at 123.19 143.51)
+		(diameter 0)
+		(color 0 0 0 0)
 	)
 	(junction
@@
 	)
 	(junction
+		(at 125.73 140.97)
+		(diameter 0)
+		(color 0 0 0 0)
+	)
+	(junction
 		(at 367.03 77.47)
 		(diameter 0)
@@
 	)
 	(junction
-		(at 73.66 224.79)
-		(diameter 0)
-		(color 0 0 0 0)
-	)
-	(junction
 		(at 336.55 135.89)
 		(diameter 0)
@@
 	)
 	(junction
-		(at 83.82 224.79)
-		(diameter 0)
-		(color 0 0 0 0)
-	)
-	(junction
 		(at 303.53 196.85)
 		(diameter 0)
@@
 	(wire
 		(pts
-			(xy 125.73 143.51) (xy 129.54 143.51)
-		)
-		(stroke
-			(width 0)
-			(type default)
-		)
-	)
-	(wire
-		(pts
 			(xy 304.8 223.52) (xy 275.59 223.52)
 		)
@@
 	(wire
 		(pts
-			(xy 208.28 203.2) (xy 208.28 199.39)
+			(xy 125.73 140.97) (xy 129.54 140.97)
 		)
 		(stroke
@@
 	(wire
 		(pts
-			(xy 205.74 205.74) (xy 205.74 199.39)
-		)
-		(stroke
-			(width 0)
-			(type default)
-		)
-	)
-	(wire
-		(pts
 			(xy 251.46 208.28) (xy 251.46 259.08)
 		)
@@
 	(wire
 		(pts
-			(xy 73.66 224.79) (xy 83.82 224.79)
-		)
-		(stroke
-			(width 0)
-			(type default)
-		)
-	)
-	(wire
-		(pts
 			(xy 96.52 48.26) (xy 96.52 57.15)
 		)
@@
 	(wire
 		(pts
+			(xy 123.19 143.51) (xy 123.19 140.97)
+		)
+		(stroke
+			(width 0)
+			(type default)
+		)
+	)
+	(wire
+		(pts
 			(xy 307.34 53.34) (xy 307.34 58.42)
 		)
@@
 	(wire
 		(pts
-			(xy 275.59 205.74) (xy 205.74 205.74)
+			(xy 275.59 205.74) (xy 208.28 205.74)
 		)
 		(stroke
@@
 	(wire
 		(pts
-			(xy 123.19 140.97) (xy 129.54 140.97)
-		)
-		(stroke
-			(width 0)
-			(type default)
-		)
-	)
-	(wire
-		(pts
 			(xy 80.01 64.77) (xy 80.01 63.5)
 		)
@@
 	(wire
 		(pts
-			(xy 125.73 160.02) (xy 125.73 143.51)
+			(xy 125.73 160.02) (xy 125.73 140.97)
 		)
 		(stroke
@@
 	(wire
 		(pts
+			(xy 205.74 203.2) (xy 205.74 199.39)
+		)
+		(stroke
+			(width 0)
+			(type default)
+		)
+	)
+	(wire
+		(pts
 			(xy 339.09 148.59) (xy 339.09 138.43)
 		)
@@
 	(wire
 		(pts
+			(xy 123.19 143.51) (xy 129.54 143.51)
+		)
+		(stroke
+			(width 0)
+			(type default)
+		)
+	)
+	(wire
+		(pts
 			(xy 259.08 215.9) (xy 200.66 215.9)
 		)
@@
 	(wire
 		(pts
+			(xy 125.73 140.97) (xy 125.73 139.7)
+		)
+		(stroke
+			(width 0)
+			(type default)
+		)
+	)
+	(wire
+		(pts
 			(xy 246.38 254) (xy 256.54 254)
 		)
@@
 	(wire
 		(pts
-			(xy 123.19 147.32) (xy 123.19 140.97)
+			(xy 123.19 147.32) (xy 123.19 143.51)
 		)
 		(stroke
@@
 	(wire
 		(pts
-			(xy 208.28 203.2) (xy 279.4 203.2)
-		)
-		(stroke
-			(width 0)
-			(type default)
-		)
-	)
-	(wire
-		(pts
 			(xy 304.8 80.01) (xy 307.34 80.01)
 		)
@@
 	(wire
 		(pts
+			(xy 205.74 203.2) (xy 279.4 203.2)
+		)
+		(stroke
+			(width 0)
+			(type default)
+		)
+	)
+	(wire
+		(pts
 			(xy 215.9 245.11) (xy 222.25 245.11)
 		)
@@
 	(wire
 		(pts
+			(xy 208.28 199.39) (xy 208.28 205.74)
+		)
+		(stroke
+			(width 0)
+			(type default)
+		)
+	)
+	(wire
+		(pts
 			(xy 213.36 264.16) (xy 251.46 264.16)
 		)
@@
 			(width 0)
 			(type default)
+		)
+	)
+	(label "XIN"
+		(at 109.22 160.02 0)
+		(effects
+			(font
+				(size 1.27 1.27)
+			)
+			(justify left bottom)
 		)
 	)
@@
 		)
 	)
+	(label "XOUT"
+		(at 109.22 147.32 0)
+		(effects
+			(font
+				(size 1.27 1.27)
+			)
+			(justify left bottom)
+		)
+	)
 	(label "SCL"
 		(at 128.27 232.41 0)
@@
 		)
 	)
-	(label "XIN"
-		(at 105.41 147.32 0)
-		(effects
-			(font
-				(size 1.27 1.27)
-			)
-			(justify left bottom)
-		)
-	)
 	(label "Photo1"
 		(at 130.81 48.26 0)
@@
 	(label "P12"
 		(at 246.38 248.92 0)
-		(effects
-			(font
-				(size 1.27 1.27)
-			)
-			(justify left bottom)
-		)
-	)
-	(label "XOUT"
-		(at 105.41 160.02 0)
 		(effects
 			(font
@@
 		(length 2.54)
 		(shape round)
-		(at 125.73 143.51 0)
+		(at 66.04 224.79 0)
 		(fields_autoplaced yes)
 		(effects
@@
 			(justify left bottom)
 		)
-		(property "Netclass" "MCU"
-			(at 126.4285 140.97 0)
+		(property "Netclass" "senyal"
+			(at 66.7385 222.25 0)
 			(effects
 				(font
@@
 				)
 				(justify left)
+				(hide yes)
 			)
 		)
 		(property "Component Class" ""
-			(at -204.47 -60.96 0)
+			(at -273.05 85.09 0)
 			(effects
 				(font
+					(size 1.27 1.27)
+					(italic yes)
+				)
+			)
+		)
+	)
+	(netclass_flag ""
+		(length 2.54)
+		(shape round)
+		(at 125.73 139.7 0)
+		(fields_autoplaced yes)
+		(effects
+			(font
+				(size 1.27 1.27)
+			)
+			(justify left bottom)
+		)
+		(property "Netclass" "MCU"
+			(at 126.4285 137.16 0)
+			(effects
+				(font
+					(size 1.27 1.27)
+				)
+				(justify left)
+			)
+		)
+		(property "Component Class" ""
+			(at -204.47 -64.77 0)
+			(effects
+				(font

Commit message: Desacoplos y limitador
Parts:
- added C6: 100n, Capacitor_SMD:C_0805_2012Metric_Pad1.18x1.45mm_HandSolder, symbol Device:C
- added R1: 1k, symbol Device:R
Connections:
- net +3.3V: now also IC1.6 (DVCC), C6.2
- net GND: now also IC1.7 (DVSS), RV1.2, RV2.2, C6.1, R1.2; no longer LCD1.7 (K)
- net Photo1: now also RV2.1; no longer RV2.2
- net Photo2: now also RV1.1; no longer RV1.2
- net Pantalla_LCD: now reaches JP1.1 (A), LCD1.6 (A)
- new net: LCD1.7 (K), R1.1
- no-connect marks 41 -> 37

Commit message: Errores layout
Parts:
- removed TP14, TP15, TP17, TP18, TP6: TestPoint, Connector_PinHeader_2.54mm:PinHeader_1x01_P2.54mm_Vertical, symbol Connector:TestPoint
- added C7: 100n, Capacitor_SMD:C_0805_2012Metric_Pad1.18x1.45mm_HandSolder, symbol Device:C
- R1: footprint (none) -> Resistor_SMD:R_0805_2012Metric_Pad1.20x1.40mm_HandSolder
- R10, R9: footprint Connector_PinHeader_2.54mm:PinHeader_1x02_P2.54mm_Horizontal -> Connector_PinHeader_2.54mm:PinHeader_1x02_P2.54mm_Vertical
Connections:
- net +3.3V: now also C7.1
- net GND: now also C7.2

Commit message: Placa acabada
Parts:
- removed C3: 100n, Capacitor_SMD:C_0805_2012Metric_Pad1.18x1.45mm_HandSolder, symbol Device:C
Changed lines of the file:
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@@
 	)
 	(junction
-		(at 38.1 219.71)
-		(diameter 0)
-		(color 0 0 0 0)
-	)
-	(junction
 		(at 80.01 63.5)
 		(diameter 0)
@@
 	(wire
 		(pts
-			(xy 38.1 220.98) (xy 38.1 219.71)
-		)
-		(stroke
-			(width 0)
-			(type default)
-		)
-	)
-	(wire
-		(pts
 			(xy 114.3 135.89) (xy 114.3 130.81)
 		)
@@
 	)
 	(symbol
-		(lib_id "power:GND")
-		(at 38.1 228.6 0)
-		(unit 1)
-		(exclude_from_sim no)
-		(in_bom yes)
-		(on_board yes)
-		(dnp no)
-		(fields_autoplaced yes)
-		(property "Reference" "#PWR09"
-			(at 38.1 234.95 0)
-			(effects
-				(font
-					(size 1.27 1.27)
-				)
-				(hide yes)
-			)
-		)
-		(property "Value" "GND"
-			(at 38.1 233.68 0)
-			(effects
-				(font
-					(size 1.27 1.27)
-				)
-			)
-		)
-		(property "Footprint" ""
-			(at 38.1 228.6 0)
-			(effects
-				(font
-					(size 1.27 1.27)
-				)
-				(hide yes)
-			)
-		)
-		(property "Datasheet" ""
-			(at 38.1 228.6 0)
-			(effects
-				(font
-					(size 1.27 1.27)
-				)
-				(hide yes)
-			)
-		)
-		(property "Description" "Power symbol creates a global label with name \"GND\" , ground"
-			(at 38.1 228.6 0)
-			(effects
-				(font
-					(size 1.27 1.27)
-				)
-				(hide yes)
-			)
-		)
-		(pin "1"
-		)
-		(instances
-			(project "placa_robot"
-				(path "/8aa50d15-d96a-41b3-aa5f-664bff39212d"
-					(reference "#PWR09")
-					(unit 1)
-				)
-			)
-		)
-	)
-	(symbol
 		(lib_id "Switch:SW_Push")
 		(at 86.36 121.92 0)
@@
 					(unit 1)
 				)
-			)
-		)
-	)
-	(symbol
-		(lib_id "Device:C")
-		(at 38.1 224.79 0)
-		(unit 1)
-		(exclude_from_sim no)
-		(in_bom yes)
-		(on_board yes)
-		(dnp no)
-		(fields_autoplaced yes)
-		(property "Reference" "C3"
-			(at 41.91 223.5199 0)
-			(effects
-				(font
-					(size 1.27 1.27)
-				)
-				(justify left)
-			)
-		)
-		(property "Value" "100n"
-			(at 41.91 226.0599 0)
-			(effects
-				(font
-					(size 1.27 1.27)
-				)
-				(justify left)
-			)
-		)
-		(property "Footprint" "Capacitor_SMD:C_0805_2012Metric_Pad1.18x1.45mm_HandSolder"
-			(at 39.0652 228.6 0)
-			(effects
-				(font
-					(size 1.27 1.27)
-				)
-				(hide yes)
-			)
-		)
-		(property "Datasheet" "~"
-			(at 38.1 224.79 0)
-			(effects
-				(font
-					(size 1.27 1.27)
-				)
-				(hide yes)
-			)
-		)
-		(property "Description" "Unpolarized capacitor"
-			(at 38.1 224.79 0)
-			(effects
-				(font
-					(size 1.27 1.27)
-				)
-				(hide yes)
-			)
-		)
-		(pin "1"
-		)
-		(pin "2"
-		)
-		(instances
-			(project "placa_robot"
-				(path "/8aa50d15-d96a-41b3-aa5f-664bff39212d"
-					(reference "C3")
-					(unit 1)
-				)
