File: placa_robot/placa_robot.kicad_pcb (KiCad board)
At the start: 2 copper layers, 80 x 75 mm, 5 parts

Commit message: Layout sin micro
Parts:
- added C2: 18p, Capacitor_SMD:C_0805_2012Metric_Pad1.18x1.45mm_HandSolder, F.Cu at (228.0, 146.0)
- added C3: 100n, Capacitor_SMD:C_0805_2012Metric_Pad1.18x1.45mm_HandSolder, F.Cu at (246.3, 79.2)
- added C4: 18p, Capacitor_SMD:C_0805_2012Metric_Pad1.18x1.45mm_HandSolder, F.Cu at (211.5, 147.0)
- added C5: 1nF, Capacitor_SMD:C_0805_2012Metric_Pad1.18x1.45mm_HandSolder, F.Cu at (166.0, 68.0)
- added J1: Conn_01x03, Connector_PinHeader_2.54mm:PinHeader_1x03_P2.54mm_Vertical, F.Cu at (162.5, 62.0)
- added J3: Conn_02x04_Odd_Even, Connector_PinHeader_2.54mm:PinHeader_2x04_P2.54mm_Vertical, F.Cu at (125.0, 61.4)
- added JP1: Jumper_2_Bridged, TestPoint:TestPoint_2Pads_Pitch2.54mm_Drill0.8mm, F.Cu at (237.8, 128.5)
- added LCD1: LCD_2x16_I2C, Connector_PinHeader_2.54mm:PinHeader_1x02_P2.54mm_Horizontal, F.Cu at (201.1, 48.2)
- added R10: R_Photo, Connector_PinHeader_2.54mm:PinHeader_1x02_P2.54mm_Horizontal, F.Cu at (121.5, 123.0)
- added R13: 10k, Resistor_SMD:R_0805_2012Metric_Pad1.20x1.40mm_HandSolder, F.Cu at (229.5, 97.0)
- added R14: 10k, Resistor_SMD:R_0805_2012Metric_Pad1.20x1.40mm_HandSolder, F.Cu at (222.9, 98.0)
- added R15: 10k, Resistor_SMD:R_0805_2012Metric_Pad1.20x1.40mm_HandSolder, F.Cu at (131.0, 65.5)
- added R16: 47k, Resistor_SMD:R_0805_2012Metric_Pad1.20x1.40mm_HandSolder, F.Cu at (166.0, 63.5)
- added R4: 1K, Resistor_SMD:R_0805_2012Metric_Pad1.20x1.40mm_HandSolder, F.Cu at (155.0, 55.5)
- added R5: 1K, Resistor_SMD:R_0805_2012Metric_Pad1.20x1.40mm_HandSolder, F.Cu at (149.5, 55.5)
- added R6: 1K, Resistor_SMD:R_0805_2012Metric_Pad1.20x1.40mm_HandSolder, F.Cu at (147.0, 59.5)
- added R9: R_Photo, Connector_PinHeader_2.54mm:PinHeader_1x02_P2.54mm_Horizontal, F.Cu at (168.3, 122.0)
- added TP1: TestPoint, Connector_PinHeader_2.54mm:PinHeader_1x01_P2.54mm_Vertical, F.Cu at (261.1, 25.2)
- added TP10: TestPoint, Connector_PinHeader_2.54mm:PinHeader_1x01_P2.54mm_Vertical, F.Cu at (120.5, 61.5)
- added TP11: TestPoint, Connector_PinHeader_2.54mm:PinHeader_1x01_P2.54mm_Vertical, F.Cu at (265.7, 29.9)
- added TP12: TestPoint, Connector_PinHeader_2.54mm:PinHeader_1x01_P2.54mm_Vertical, F.Cu at (265.7, 34.5)
- added TP13: TestPoint, Connector_PinHeader_2.54mm:PinHeader_1x01_P2.54mm_Vertical, F.Cu at (127.5, 74.0)
- added TP14: TestPoint, Connector_PinHeader_2.54mm:PinHeader_1x01_P2.54mm_Vertical, F.Cu at (270.4, 29.9)
- added TP15: TestPoint, Connector_PinHeader_2.54mm:PinHeader_1x01_P2.54mm_Vertical, F.Cu at (270.4, 34.5)
- added TP16: TestPoint, Connector_PinHeader_2.54mm:PinHeader_1x01_P2.54mm_Vertical, F.Cu at (275.0, 25.2)
- added TP17: TestPoint, Connector_PinHeader_2.54mm:PinHeader_1x01_P2.54mm_Vertical, F.Cu at (275.0, 29.9)
- added TP18: TestPoint, Connector_PinHeader_2.54mm:PinHeader_1x01_P2.54mm_Vertical, F.Cu at (275.0, 34.5)
- added TP2: TestPoint, Connector_PinHeader_2.54mm:PinHeader_1x01_P2.54mm_Vertical, F.Cu at (261.1, 29.9)
- added TP6: TestPoint, Connector_PinHeader_2.54mm:PinHeader_1x01_P2.54mm_Vertical, F.Cu at (261.1, 34.5)
- added U1: LM324, Package_SO:SOIC-14_3.9x8.7mm_P1.27mm, F.Cu at (145.5, 67.0)
- added Y1: Crystal, Crystal:Crystal_DS26_D2.0mm_L6.0mm_Horizontal, F.Cu at (218.1, 141.0)
- moved REF** 76.0 mm to (176.0, 120.0), turned to 90 degrees
- moved REF** 68.2 mm to (110.0, 120.0), turned to 90 degrees
- moved REF** 47.9 mm to (143.5, 49.0), turned to 90 degrees
- moved REF** 43.9 mm to (168.5, 79.5), turned to 90 degrees
- moved REF** 31.4 mm to (117.0, 79.5), turned to 90 degrees
Routing:
- net Net-(U1C--): track 0.00 -> 10.2 mm
- net Net-(S2-2'): track 0.00 -> 9.09 mm
- net /LSB: track 0.00 -> 7.99 mm
- net /MSB: track 0.00 -> 7.56 mm, vias 0 -> 2
- net GND: track 0.00 -> 6.91 mm, vias 0 -> 3
- net +3.3V: track 0.00 -> 6.56 mm, vias 0 -> 3
- net /MCU_RST: track 0.00 -> 5.98 mm
- net /WIFI_TXD: track 0.00 -> 4.96 mm
- net /WIFI_RXD: track 0.00 -> 4.49 mm
- net Net-(J3-Pin_6): track 0.00 -> 3.50 mm
- added copper zone on F.Cu, net +3.3V
- added copper zone on B.Cu, net GND
Other:
- board size 80 x 75 mm -> 75 x 80 mm

Commit message: Progreso actual Layout y errores
Parts:
- removed REF** (x5): MountingHole_3.2mm_M3, MountingHole:MountingHole_3.2mm_M3
- added IC1: MSP430FR2355TPT, MiSE:QFP50P900X900X160-48N, F.Cu at (143.8, 93.8)
- added J4: conn_DFrobot, MiSE:conn_DFrobot, F.Cu at (142.9, 109.0)
- added RV1: R_POT, MiSE:Trimmer_MiSE, F.Cu at (23.8, 188.8)
- added RV2: R_POT, MiSE:Trimmer_MiSE, F.Cu at (31.9, 188.8)
- LCD1: footprint Connector_PinHeader_2.54mm:PinHeader_1x02_P2.54mm_Horizontal -> MiSE:LCD_2x16_I2C(Midas)
- moved J3 83.0 mm to (206.5, 76.9)
- moved R15 83.0 mm to (212.5, 81.0)
- moved TP10 83.0 mm to (202.0, 77.0)
- moved TP13 83.0 mm to (209.0, 89.5)
- moved LCD1 77.1 mm to (147.0, 103.1)
- moved R10 73.7 mm to (108.5, 50.5), turned to 90 degrees
- moved R9 72.9 mm to (174.7, 49.4), turned to 90 degrees
Routing:
- net /WIFI_TXD: track 4.96 -> 0.00 mm
- net +3.3V: track 6.56 -> 2.03 mm, vias 3 -> 1
- net /WIFI_RXD: track 4.49 -> 0.11 mm
- net Net-(J3-Pin_6): track 3.50 -> 0.00 mm

Commit message: Cambios layout
Parts:
- added J2: Conn_01x01, Connector_PinHeader_2.54mm:PinHeader_1x01_P2.54mm_Vertical, F.Cu at (169.0, 118.0)
- added S2: THB001P, MiSE:THB001P, F.Cu at (139.8, 99.2)
- added SW1: SW_Push, Button_Switch_THT:SW_PUSH_6mm, F.Cu at (175.2, 99.2)
- moved RV1 145.8 mm to (126.9, 85.8)
- moved RV2 145.8 mm to (135.0, 85.8)
- moved C2 112.7 mm to (148.0, 66.5), turned to -90 degrees
- moved C4 101.3 mm to (150.0, 66.5), turned to -90 degrees
- moved Y1 100.1 mm to (148.1, 69.5)
- moved J3 99.9 mm to (110.5, 104.4)
- moved R15 97.7 mm to (117.5, 104.0)
- moved R10 95.2 mm to (179.0, 114.5), turned to -90 degrees
- moved R9 90.5 mm to (113.5, 116.0), turned to -90 degrees
- moved JP1 78.6 mm to (159.8, 118.5)
- moved TP14 77.2 mm to (204.3, 69.8)
- moved TP15 77.2 mm to (204.3, 74.5)
- moved TP1 77.2 mm to (195.1, 65.2)
- moved TP11 77.2 mm to (199.7, 69.8)
- moved TP12 77.2 mm to (199.7, 74.5)
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Connections:
- IC1 pad 42: /Photo1 -> /Photo2
- IC1 pad 43: /Photo2 -> /Photo1
- IC1 pad 45: /DOWN -> /UP
- IC1 pad 46: /UP -> /DOWN
Routing:
- net /SCL: track 0.00 -> 80.2 mm, vias 0 -> 2
- net /SDA: track 0.00 -> 80.2 mm
- net /Photo1: track 0.04 -> 78.3 mm
- net /MCU_RST: track 5.98 -> 81.0 mm
- net /SBW: track 0.00 -> 66.8 mm
- net /JOY_BOTTON: track 0.00 -> 63.5 mm, vias 0 -> 2
- net /WIFI_TXD: track 0.00 -> 63.4 mm, vias 0 -> 2
- net /Photo2: track 0.00 -> 61.8 mm
- net /WIFI_RXD: track 0.11 -> 50.5 mm
- net /LCD_RST: track 0.00 -> 30.8 mm, vias 0 -> 2
- net /DOWN: track 0.00 -> 29.2 mm
- net Net-(U1C--): track 10.2 -> 36.0 mm
- net /RIGHT: track 0.00 -> 20.6 mm, vias 0 -> 2
- net /P0: track 0.00 -> 17.3 mm
- net /P1: track 0.00 -> 15.7 mm
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Other:
- board text added: "Universidad de Barcelona - 2026 Alex Yang & Eric trejo"

Commit message: cambio layout
Parts:
- removed TP1, TP10, TP11, TP12, TP13, TP14, TP15, TP16, TP17, TP18, TP2, TP6: TestPoint, Connector_PinHeader_2.54mm:PinHeader_1x01_P2.54mm_Vertical
- moved JP1 53.8 mm to (179.0, 68.2), turned to 90 degrees
- moved C2 14.0 mm to (162.0, 67.3)
- moved C4 14.0 mm to (164.0, 67.3)
- moved Y1 0.89 mm to (147.5, 70.2), turned to 90 degrees
Connections:
- C2 pad 2: /XOUT -> Net-(IC1-P2.7/TB0CLK/XIN)
- C4 pad 2: /XIN -> Net-(IC1-P2.6/MCLK/XOUT)
- IC1 pad 23: /WIFI_TXD -> /WIFI_RXD
- IC1 pad 24: /WIFI_RXD -> /WIFI_TXD
- IC1 pad 8: /XIN -> Net-(IC1-P2.7/TB0CLK/XIN)
- IC1 pad 9: /XOUT -> Net-(IC1-P2.6/MCLK/XOUT)
- Y1 pad 1: /XOUT -> Net-(IC1-P2.7/TB0CLK/XIN)
- Y1 pad 2: /XIN -> Net-(IC1-P2.6/MCLK/XOUT)
Routing:
- net /WIFI_RXD: track 50.5 -> 60.2 mm
- net /XIN: track 8.18 -> 0.00 mm
- net /XOUT: track 5.86 -> 0.00 mm
- net /WIFI_TXD: track 63.4 -> 61.6 mm, vias 2 -> 0
- net /DOWN: track 29.2 -> 29.9 mm
